File: PCB/robarm_kicad/robarm_kicad.kicad_sch (KiCad schematic)
At the start: 0 parts

Commit message: got the motor control working in ONE direction. the other direction is still not working. ADC still not working
Parts:
- added J1, J2, J3, J4, J5, J6: Conn_01x05_Pin, Connector_JST:JST_XH_B5B-XH-A_1x05_P2.50mm_Vertical, symbol Connector:Conn_01x05_Pin
- added J7: Barrel_Jack_MountingPin, Connector_BarrelJack:BarrelJack_Horizontal, symbol Connector:Barrel_Jack_MountingPin
- added U1: STM32F411 BlackPill, WeAct_Black_Pill_V2.0:STM32F411_Black_Pill, symbol WeAct_Black_Pill_V2.0:STM32F411_Black_Pill
- added U2, U3, U4: ROB-14450, ROB-14450:MODULE_ROB-14450, symbol ROB-14450:ROB-14450
- added U5: L7805, Package_TO_SOT_THT:TO-220-3_Horizontal_TabDown, symbol Regulator_Linear:L7805
Connections:
- new net 12v: J7.1, U2.1 (VM), U3.1 (VM), U4.1 (VM), U5.1 (IN)
- new net 3v3: J1.3 (Pin_3), J2.3 (Pin_3), J3.3 (Pin_3), J4.3 (Pin_3), J5.3 (Pin_3), J6.3 (Pin_3), U1.38 (3.3V)
- new net 5v: U1.40 (5V), U2.2 (VCC), U3.2 (VCC), U4.2 (VCC), U5.3 (OUT)
- new net A01: U1.23 (C14), U2.14 (AI1)
- new net A02: U1.24 (C15), U2.15 (AI2)
- new net A11: U1.36 (B2), U3.14 (AI1)
- new net A12: U1.37 (B10), U3.15 (AI2)
- new net A21: U1.6 (A9), U4.14 (AI1)
- new net A22: U1.5 (A8), U4.15 (AI2)
- new net B01: U1.11 (B3), U2.12 (BI1)
- new net B02: U1.10 (A15), U2.11 (BI2)
- new net B11: U1.35 (B1), U3.12 (BI1)
- new net B12: U1.34 (B0), U3.11 (BI2)
- new net B21: U1.4 (B15), U4.12 (BI1)
- new net B22: U1.33 (A7), U4.11 (BI2)
- new net GND: J1.4 (Pin_4), J2.4 (Pin_4), J3.4 (Pin_4), J4.4 (Pin_4), J5.4 (Pin_4), J6.4 (Pin_4), J7.2, J7.MP (MountPin), U1.19 (G), U1.39 (G), U2.3 (GND), U2.8 (GND), U2.9 (GND), U3.3 (GND), U3.8 (GND), U3.9 (GND), U4.3 (GND), U4.8 (GND), U4.9 (GND), U5.2 (GND)
- new net MA0N: J1.2 (Pin_2), U2.5 (A02)
- new net MA0P: J1.1 (Pin_1), U2.4 (A01)
- new net MA1N: J3.2 (Pin_2), U3.5 (A02)
- new net MA1P: J3.1 (Pin_1), U3.4 (A01)
- new net MA2N: J5.2 (Pin_2), U4.5 (A02)
- new net MA2P: J5.1 (Pin_1), U4.4 (A01)
- new net MB0N: J2.2 (Pin_2), U2.6 (B02)
- new net MB0P: J2.1 (Pin_1), U2.7 (B01)
- new net MB1N: J4.2 (Pin_2), U3.6 (B02)
- new net MB1P: J4.1 (Pin_1), U3.7 (B01)
- new net MB2N: J6.2 (Pin_2), U4.6 (B02)
- new net MB2P: J6.1 (Pin_1), U4.7 (B01)
- new net encA0: J1.5 (Pin_5), U1.27 (A1)
- new net encA1: J3.5 (Pin_5), U1.29 (A3)
- new net encA2: J5.5 (Pin_5), U1.31 (A5)
- new net encB0: J2.5 (Pin_5), U1.28 (A2)
- new net encB1: J4.5 (Pin_5), U1.30 (A4)
- new net encB2: J6.5 (Pin_5), U1.32 (A6)
- new net pwmA0: U1.17 (B9), U2.16 (PWMA)
- new net pwmA1: U1.15 (B7), U3.16 (PWMA)
- new net pwmA2: U1.13 (B5), U4.16 (PWMA)
- new net pwmB0: U1.16 (B8), U2.10 (PWMB)
- new net pwmB1: U1.14 (B6), U3.10 (PWMB)
- new net pwmB2: U1.12 (B4), U4.10 (PWMB)
- new net stby0: U1.1 (B12), U2.13 (STBY)
- new net stby1: U1.2 (B13), U3.13 (STBY)
- new net stby2: U1.3 (B14), U4.13 (STBY)
- no-connect marks 0 -> 9
